File: dual-sx1281-carrier-board/dual-sx1281-carrier-board.kicad_pcb (KiCad board)
At the start: 2 copper layers, 68.8 x 34.3 mm, 28 parts, among them J1 Conn_01x05, J2 Conn_01x04_Pin, J3 Conn_01x04_Pin, J4 Conn_01x04_Pin, J5 Conn_01x04_Pin, U1 RP2040, U2 W25Q32JVSS, U3 E28-2G4M20SX, U4 E28-2G4M20SX, Y1 Crystal_GND24

Commit message: Mouting-holes
Parts:
- added H1: MountingHole, MountingHole:MountingHole_2mm, F.Cu at (147.9, 87.9)
- added H2: MountingHole, MountingHole:MountingHole_2mm, F.Cu at (209.7, 87.9)
- added H3: MountingHole, MountingHole:MountingHole_2mm, F.Cu at (147.9, 115.8)
- added H4: MountingHole, MountingHole:MountingHole_2mm, F.Cu at (209.7, 115.8)
- R1, R2: footprint Resistor_SMD:R_0201_0603Metric -> Resistor_SMD:R_0402_1005Metric
- R4: footprint Resistor_SMD:R_0201_0603Metric -> Resistor_SMD:R_0603_1608Metric
- moved U3 45.3 mm to (156.0, 101.0)
- moved U4 44.3 mm to (201.0, 101.0)
- moved J2 35.1 mm to (175.0, 119.0), turned to 90 degrees
- moved J3 35.1 mm to (182.6, 84.7), turned to -90 degrees
- moved R1 19.8 mm to (167.7, 92.1), turned to -90 degrees
- moved J1 19.1 mm to (171.4, 112.5), turned to 0 degrees
- moved C14 19.1 mm to (189.0, 109.4), turned to 0 degrees
- moved Y1 16.4 mm to (185.4, 110.3), turned to 0 degrees
- moved C13 15.2 mm to (181.7, 111.3), turned to 180 degrees
- moved C8 15.1 mm to (188.2, 106.3), turned to 0 degrees
- moved C4 14.3 mm to (188.5, 104.7), turned to 0 degrees
- moved R4 14.2 mm to (188.4, 101.5), turned to -90 degrees
- moved C1 13.9 mm to (175.0, 91.8), turned to 90 degrees
- moved R2 13.2 mm to (186.1, 106.8), turned to -90 degrees
- moved U2 12.4 mm to (171.2, 96.1), turned to 0 degrees
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Connections:
- net Net-(J1-Pin_1) renamed /SWCLK
- net Net-(J1-Pin_2) renamed /SWDIO
- net Net-(U1-RUN) renamed /RUN
- U1 pad 11: unconnected-(U1-GPIO8-Pad11) -> /LORA1 NRST
- U1 pad 12: unconnected-(U1-GPIO9-Pad12) -> /LORA1_TX_EN
- U1 pad 13: unconnected-(U1-GPIO10-Pad13) -> /LORA1_RX_EN
- U1 pad 31: /SPI0 RX -> unconnected-(U1-GPIO20-Pad31)
- U1 pad 32: /SPI0 CS -> unconnected-(U1-GPIO21-Pad32)
- U1 pad 34: /SPI0 SCK -> unconnected-(U1-GPIO22-Pad34)
- U1 pad 35: /SPI0 TX -> unconnected-(U1-GPIO23-Pad35)
- U1 pad 36: /LORA1 IRQ -> unconnected-(U1-GPIO24-Pad36)
- U1 pad 37: /LORA1 BUSY -> unconnected-(U1-GPIO25-Pad37)
- U1 pad 38: /LORA1 NRST -> unconnected-(U1-GPIO26/ADC0-Pad38)
- U1 pad 39: /LORA1_TX_EN -> unconnected-(U1-GPIO27/ADC1-Pad39)
- U1 pad 4: unconnected-(U1-GPIO2-Pad4) -> /SPI0 SCK
- U1 pad 40: /LORA1_RX_EN -> unconnected-(U1-GPIO28/ADC2-Pad40)
- U1 pad 5: unconnected-(U1-GPIO3-Pad5) -> /SPI0 TX
- U1 pad 6: unconnected-(U1-GPIO4-Pad6) -> /SPI0 RX
- U1 pad 7: unconnected-(U1-GPIO5-Pad7) -> /SPI0 CS
- U1 pad 8: unconnected-(U1-GPIO6-Pad8) -> /LORA1 IRQ
- U1 pad 9: unconnected-(U1-GPIO7-Pad9) -> /LORA1 BUSY
Routing:
- net +3V3: track 115.5 -> 42.2 mm
- net /LORA1_RX_EN: track 0.00 -> 36.7 mm
- net GND: track 12.1 -> 40.4 mm, vias 51 -> 34
- net /LORA1 IRQ: track 37.6 -> 19.5 mm, vias 2 -> 0
- net /LORA2 BUSY: track 42.6 -> 24.9 mm, vias 4 -> 2
- net +1V1: track 8.41 -> 25.9 mm, vias 0 -> 4
- net /LORA1 BUSY: track 38.1 -> 20.8 mm
- net /SPI0 TX: track 19.7 -> 36.8 mm, vias 0 -> 2
- net /LORA1 NRST: track 38.0 -> 22.3 mm
- net /LORA1_TX_EN: track 36.8 -> 21.6 mm
- net /LORA2 IRQ: track 40.2 -> 25.4 mm, vias 4 -> 2
- net /SPI0 CS: track 21.2 -> 34.1 mm, vias 2 -> 0
- net /SPI0 SCK: track 20.2 -> 32.1 mm, vias 0 -> 2
- net /SPI1 CS: track 26.7 -> 16.0 mm
- net /SPI0 RX: track 29.1 -> 39.6 mm
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- added copper zone on F.Cu, net +3V3
- added copper zone on In2.Cu, net GND
Other:
- copper layers 2 -> 4

Commit message: PCB fully routed
Parts:
- added D1: LED, LED_SMD:LED_0603_1608Metric, F.Cu at (191.3, 87.2)
- added D2: LED, LED_SMD:LED_0603_1608Metric, F.Cu at (188.7, 87.2)
- added D3: LED, LED_SMD:LED_0603_1608Metric, F.Cu at (186.1, 87.2)
- added R5: 300, Resistor_SMD:R_0603_1608Metric, F.Cu at (191.3, 91.2)
- added R6: 300, Resistor_SMD:R_0603_1608Metric, F.Cu at (188.8, 91.2)
- added R7: 300, Resistor_SMD:R_0603_1608Metric, F.Cu at (186.3, 91.2)
- moved C10 1.01 mm to (186.2, 96.2)
Connections:
- J3 pad 2: GND -> /IO1
- J3 pad 3: GND -> /IO2
- J3 pad 4: GND -> +3V3
- U1 pad 31: unconnected-(U1-GPIO20-Pad31) -> /LED_R
- U1 pad 32: unconnected-(U1-GPIO21-Pad32) -> /LED_G
- U1 pad 34: unconnected-(U1-GPIO22-Pad34) -> /LED_B
- U1 pad 35: unconnected-(U1-GPIO23-Pad35) -> /IO1
- U1 pad 36: unconnected-(U1-GPIO24-Pad36) -> /IO2
Routing:
- net /IO2: track 0.00 -> 17.6 mm
- net /IO1: track 0.00 -> 17.0 mm
- net /LED_R: track 0.00 -> 11.4 mm
- net /LED_G: track 0.00 -> 10.2 mm
- net /LED_B: track 0.00 -> 8.83 mm
- net +3V3: track 42.2 -> 47.8 mm
- net /SPI1 CLK: track 22.9 -> 18.1 mm
- net /SPI0 RX: track 39.6 -> 37.1 mm
- net Net-(D3-K): track 0.00 -> 2.48 mm
- net Net-(D2-K): track 0.00 -> 2.45 mm
- net Net-(D1-K): track 0.00 -> 2.41 mm
- net /SPI0 TX: track 36.8 -> 34.8 mm
- net /SPI0 CS: track 34.1 -> 34.7 mm
- net /RX0: track 21.0 -> 21.2 mm, vias 2 -> 3
- net /TX0: vias 2 -> 3

Commit message: Silkscreen and nice PCB image for docs
Parts:
- removed J1: Conn_01x05, Connector_Molex:Molex_PicoBlade_53398-0571_1x05-1MP_P1.25mm_Vertical
- added J6: Conn_01x06, Connector_Molex:Molex_PicoBlade_53398-0671_1x06-1MP_P1.25mm_Vertical, F.Cu at (172.1, 112.4)
Routing:
- net +3V3: track 47.8 -> 47.3 mm
Other:
- outline, holes or cut-outs redrawn
- board text added: "3V3"
- board text added: "GND"
- board text added: "IO1"
- board text added: "IO2"
- board text added: "RQ2 Telemetry V3 (c) 2026 Diez Roggisch"
- board text added: "RX"
- board text added: "SWCLK"
- board text added: "SWDIO"
- board text added: "TX"
