File: dual-sx1281-carrier-board/dual-sx1281-carrier-board.kicad_sch (KiCad schematic)
At the start: 0 parts

Commit message: Start work on software based on breadboard setup
Parts:
- added C1, C10, C11, C12, C4, C5, C6, C7, C8, C9: 0.1uF, Capacitor_SMD:C_0603_1608Metric, symbol Device:C
- added C13, C14: 27pF, Capacitor_SMD:C_0603_1608Metric, symbol Device:C
- added C2, C3: 1uF, Capacitor_SMD:C_0603_1608Metric, symbol Device:C
- added J1: Conn_01x05, Connector_Molex:Molex_PicoBlade_53398-0571_1x05-1MP_P1.25mm_Vertical, symbol Connector_Generic:Conn_01x05
- added J2, J3, J4, J5: Conn_01x04_Pin, Connector_PinHeader_2.54mm:PinHeader_1x04_P2.54mm_Vertical, symbol Connector:Conn_01x04_Pin
- added R1, R4: 10K, Resistor_SMD:R_0201_0603Metric, symbol Device:R
- added R2: 1K, Resistor_SMD:R_0201_0603Metric, symbol Device:R
- added R3: DNP, Resistor_SMD:R_0201_0603Metric, symbol Device:R
- added U1: RP2040, Package_DFN_QFN:QFN-56-1EP_7x7mm_P0.4mm_EP3.2x3.2mm, symbol MCU_RaspberryPi:RP2040
- added U2: W25Q32JVSS, Package_SO:SOIC-8_5.3x5.3mm_P1.27mm, symbol Memory_Flash:W25Q32JVSS
- added U3, U4: E28-2G4M20SX, deets:E28-2G4M20SX, symbol deets kicad lib:E28-2G4M20SX
- added Y1: Crystal_GND24, Crystal:Crystal_SMD_3225-4Pin_3.2x2.5mm, symbol Device:Crystal_GND24
Connections:
- new net: R4.2, U1.26 (RUN)
- new net: C14.1, R2.2, Y1.3
- new net: J1.1 (Pin_1), U1.24 (SWCLK)
- new net: J1.2 (Pin_2), U1.25 (SWDIO)
- new net: U1.51 (QSPI_SD3), U2.7 (~{HOLD}/~{RESET}/IO_{3})
- new net: U1.52 (QSPI_SCLK), U2.6 (CLK)
- new net: U1.53 (QSPI_SD0), U2.5 (DI/IO_{0})
- new net: U1.54 (QSPI_SD2), U2.3 (~{WP}/IO_{2})
- new net: U1.55 (QSPI_SD1), U2.2 (DO/IO_{1})
- new net: R1.2, U1.56 (~{QSPI_SS}), U2.1 (~{CS})
- new net +1V1: C3.1, C4.1, C5.1, U1.23 (DVDD), U1.45 (VREG_VOUT), U1.50 (DVDD)
- new net +3V3: C1.1, C10.1, C11.1, C12.1, C2.1, C6.1, C7.1, C8.1, C9.1, J2.4 (Pin_4), R1.1, R4.1, U1.1 (IOVDD), U1.10 (IOVDD), U1.22 (IOVDD), U1.33 (IOVDD), U1.42 (IOVDD), U1.43 (ADC_AVDD), U1.44 (VREG_VIN), U1.48 (USB_VDD), U1.49 (IOVDD), U2.8 (VCC), U3.1 (VCC), U4.1 (VCC)
- new net GND: C1.2, C10.2, C11.2, C12.2, C13.2, C14.2, C2.2, C3.2, C4.2, C5.2, C6.2, C7.2, C8.2, C9.2, J1.3 (Pin_3), J2.1 (Pin_1), J3.1 (Pin_1), J3.2 (Pin_2), J3.3 (Pin_3), J3.4 (Pin_4), J4.1 (Pin_1), J4.2 (Pin_2), J4.3 (Pin_3), J4.4 (Pin_4), J5.1 (Pin_1), J5.2 (Pin_2), J5.3 (Pin_3), J5.4 (Pin_4), U1.19 (TESTEN), U1.57 (GND), U2.4 (GND), U3.10 (GND), U3.16 (GND), U3.2 (GND), U3.7 (GND), U4.10 (GND), U4.16 (GND), U4.2 (GND), U4.7 (GND), Y1.2 (G), Y1.4 (G)
- new net LORA1 BUSY: U1.37 (GPIO25), U3.12 (BUSY)
- new net LORA1 IRQ: U1.36 (GPIO24), U3.13 (DIO1)
- new net LORA1 NRST: U1.38 (GPIO26/ADC0), U3.11 (NRST)
- new net LORA1_RX_EN: U1.40 (GPIO28/ADC2), U3.8 (RX_EN)
- new net LORA1_TX_EN: U1.39 (GPIO27/ADC1), U3.9 (TX_EN)
- new net LORA2 BUSY: U1.28 (GPIO17), U4.12 (BUSY)
- new net LORA2 IRQ: U1.27 (GPIO16), U4.13 (DIO1)
- new net LORA2 NRST: U1.29 (GPIO18), U4.11 (NRST)
- new net LORA2_RX_EN: U1.18 (GPIO15), U4.8 (RX_EN)
- new net LORA2_TX_EN: U1.30 (GPIO19), U4.9 (TX_EN)
- new net RX0: J1.5 (Pin_5), J2.3 (Pin_3), U1.3 (GPIO1)
- new net SPI0 CS: U1.32 (GPIO21), U3.6 (NSS)
- new net SPI0 RX: U1.31 (GPIO20), U3.3 (MISO)
- new net SPI0 SCK: U1.34 (GPIO22), U3.5 (SCK)
- new net SPI0 TX: U1.35 (GPIO23), U3.4 (MOSI)
- new net SPI1 CLK: U1.17 (GPIO14), U4.5 (SCK)
- new net SPI1 CS: U1.16 (GPIO13), U4.6 (NSS)
- new net SPI1 RX: U1.15 (GPIO12), U4.3 (MISO)
- new net SPI1 TX: U1.14 (GPIO11), U4.4 (MOSI)
- new net TX0: J1.4 (Pin_4), J2.2 (Pin_2), U1.2 (GPIO0)
- new net XIN: C13.1, R3.1, U1.20 (XIN), Y1.1
- new net XOUT: R2.1, R3.2, U1.21 (XOUT)
- no-connect marks 0 -> 16
Other:
- note added: "Castellations"
- note added: "Close to ADC_AVDD"
- note added: "Close to DVDD pins"
- note added: "Close to IOVDD pins"

Commit message: Mouting-holes
Parts:
- added H1, H2, H3, H4: MountingHole, MountingHole:MountingHole_2mm, symbol Mechanical:MountingHole
- R1, R2, R3: footprint Resistor_SMD:R_0201_0603Metric -> Resistor_SMD:R_0402_1005Metric
- R4: footprint Resistor_SMD:R_0201_0603Metric -> Resistor_SMD:R_0603_1608Metric
Connections:
- net LORA1 BUSY: now also U1.9 (GPIO7); no longer U1.37 (GPIO25)
- net LORA1 IRQ: now also U1.8 (GPIO6); no longer U1.36 (GPIO24)
- net LORA1 NRST: now also U1.11 (GPIO8); no longer U1.38 (GPIO26/ADC0)
- net LORA1_RX_EN: now also U1.13 (GPIO10); no longer U1.40 (GPIO28/ADC2)
- net LORA1_TX_EN: now also U1.12 (GPIO9); no longer U1.39 (GPIO27/ADC1)
- net SPI0 CS: now also U1.7 (GPIO5); no longer U1.32 (GPIO21)
- net SPI0 RX: now also U1.6 (GPIO4); no longer U1.31 (GPIO20)
- net SPI0 SCK: now also U1.4 (GPIO2); no longer U1.34 (GPIO22)
- net SPI0 TX: now also U1.5 (GPIO3); no longer U1.35 (GPIO23)
- net RUN: now reaches R4.2, U1.26 (RUN)
- net SWCLK: now reaches J1.1 (Pin_1), U1.24 (SWCLK)
- net SWDIO: now reaches J1.2 (Pin_2), U1.25 (SWDIO)

Commit message: PCB fully routed
Parts:
- added D1, D2, D3: LED, LED_SMD:LED_0603_1608Metric, symbol Device:LED
- added R5, R6, R7: 300, Resistor_SMD:R_0603_1608Metric, symbol Device:R
Connections:
- net +3V3: now also J3.4 (Pin_4), D1.2 (A), D2.2 (A), D3.2 (A)
- net GND: no longer J3.2 (Pin_2), J3.3 (Pin_3), J3.4 (Pin_4)
- net LED_R: now reaches U1.31 (GPIO20)
- net LED_R: now also R5.2
- net LED_G: now reaches U1.32 (GPIO21)
- net LED_G: now also R6.2
- net LED_B: now reaches U1.34 (GPIO22)
- net LED_B: now also R7.2
- net IO1: now reaches U1.35 (GPIO23)
- net IO1: now also J3.2 (Pin_2)
- net IO2: now reaches U1.36 (GPIO24)
- net IO2: now also J3.3 (Pin_3)
- new net: D2.1 (K), R6.1
- new net: D1.1 (K), R5.1
- new net: D3.1 (K), R7.1
- no-connect marks 16 -> 11

Commit message: Silkscreen and nice PCB image for docs
Parts:
- removed J1: Conn_01x05, Connector_Molex:Molex_PicoBlade_53398-0571_1x05-1MP_P1.25mm_Vertical, symbol Connector_Generic:Conn_01x05
- added J6: Conn_01x06, Connector_Molex:Molex_PicoBlade_53398-0671_1x06-1MP_P1.25mm_Vertical, symbol Connector_Generic:Conn_01x06
Connections:
- net +3V3: now also J6.6 (Pin_6)
- net GND: now also J6.3 (Pin_3)
- net RX0: now also J6.5 (Pin_5)
- net SWCLK: now also J6.1 (Pin_1)
- net SWDIO: now also J6.2 (Pin_2)
- net TX0: now also J6.4 (Pin_4)
Changed lines of the file:
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@@
 	(wire
 		(pts
+			(xy 102.87 142.24) (xy 102.87 148.59)
+		)
+		(stroke
+			(width 0)
+			(type default)
+		)
+	)
+	(wire
+		(pts
 			(xy 245.11 129.54) (xy 247.65 129.54)
 		)
@@
 	(wire
 		(pts
+			(xy 116.84 148.59) (xy 102.87 148.59)
+		)
+		(stroke
+			(width 0)
+			(type default)
+		)
+	)
+	(wire
+		(pts
 			(xy 27.94 39.37) (xy 27.94 41.91)
 		)
@@
 	(wire
 		(pts
+			(xy 116.84 142.24) (xy 116.84 148.59)
+		)
+		(stroke
+			(width 0)
+			(type default)
+		)
+	)
+	(wire
+		(pts
 			(xy 139.7 191.77) (xy 149.86 191.77)
 		)
@@
 	)
 	(symbol
+		(lib_id "power:+3V3")
+		(at 102.87 142.24 0)
+		(unit 1)
+		(body_style 1)
+		(exclude_from_sim no)
+		(in_bom yes)
+		(on_board yes)
+		(in_pos_files yes)
+		(dnp no)
+		(fields_autoplaced yes)
+		(property "Reference" "#PWR030"
+			(at 102.87 146.05 0)
+			(hide yes)
+			(show_name no)
+			(do_not_autoplace no)
+			(effects
+				(font
+					(size 1.27 1.27)
+				)
+			)
+		)
+		(property "Value" "+3V3"
+			(at 102.87 137.16 0)
+			(show_name no)
+			(do_not_autoplace no)
+			(effects
+				(font
+					(size 1.27 1.27)
+				)
+			)
+		)
+		(property "Footprint" ""
+			(at 102.87 142.24 0)
+			(hide yes)
+			(show_name no)
+			(do_not_autoplace no)
+			(effects
+				(font
+					(size 1.27 1.27)
+				)
+			)
+		)
+		(property "Datasheet" ""
+			(at 102.87 142.24 0)
+			(hide yes)
+			(show_name no)
+			(do_not_autoplace no)
+			(effects
+				(font
+					(size 1.27 1.27)
+				)
+			)
+		)
+		(property "Description" "Power symbol creates a global label with name \"+3V3\""
+			(at 102.87 142.24 0)
+			(hide yes)
+			(show_name no)
+			(do_not_autoplace no)
+			(effects
+				(font
+					(size 1.27 1.27)
+				)
+			)
+		)
+		(pin "1"
+		)
+		(instances
+			(project "dual-sx1281-carrier-board"
+				(path "/dd3d82ed-b0ea-48bf-93b4-f28bcc2a961e"
+					(reference "#PWR030")
+					(unit 1)
+				)
+			)
+		)
+	)
+	(symbol
 		(lib_id "power:GND")
 		(at 242.57 85.09 0)
@@
 	)
 	(symbol
-		(lib_id "deets kicad lib:E28-2G4M20SX")
-		(at 246.38 66.04 0)
+		(lib_id "Connector_Generic:Conn_01x06")
+		(at 111.76 134.62 0)
+		(mirror y)
 		(unit 1)
 		(body_style 1)
@@
 		(dnp no)
 		(fields_autoplaced yes)
-		(property "Reference" "U3"
-			(at 248.5233 50.8 0)
+		(property "Reference" "J6"
+			(at 111.76 123.19 0)
 			(show_name no)
 			(do_not_autoplace no)
@@
 					(size 1.27 1.27)
 				)
-				(justify left)
 			)
 		)
-		(property "Value" "E28-2G4M20SX"
-			(at 246.126 82.042 0)
-			(hide yes)
+		(property "Value" "Conn_01x06"
+			(at 111.76 125.73 0)
 			(show_name no)
 			(do_not_autoplace no)
@@
 			)
 		)
-		(property "Footprint" "deets:E28-2G4M20SX"
-			(at 246.126 48.514 0)
+		(property "Footprint" "Connector_Molex:Molex_PicoBlade_53398-0671_1x06-1MP_P1.25mm_Vertical"
+			(at 111.76 134.62 0)
 			(hide yes)
 			(show_name no)
@@
 		)
 		(property "Datasheet" ""
-			(at 246.38 66.04 0)
+			(at 111.76 134.62 0)
 			(hide yes)
 			(show_name no)
@@
 			)
 		)
-		(property "Description" "Lora1"
-			(at 248.5233 53.34 0)
-			(show_name no)
-			(do_not_autoplace no)
-			(effects
-				(font
-					(size 1.27 1.27)
-				)
-				(justify left)
-			)
-		)
-		(property "Manufacturer" "SenseCAP"
-			(at 246.126 51.054 0)
+		(property "Description" "Generic connector, single row, 01x06, script generated (kicad-library-utils/schlib/autogen/connector/)"
+			(at 111.76 134.62 0)
 			(hide yes)
 			(show_name no)
@@
 			)
 		)
-		(pin "15"
-		)
-		(pin "10"
-		)
-		(pin "12"
-		)
-		(pin "14"
-		)
-		(pin "13"
-		)
-		(pin "11"
+		(pin "1"
 		)
 		(pin "2"
 		)
-		(pin "16"
-		)
-		(pin "7"
-		)
-		(pin "4"
+		(pin "6"
 		)
 		(pin "3"
 		)
-		(pin "9"
-		)
-		(pin "1"
+		(pin "4"
 		)
 		(pin "5"
 		)
-		(pin "8"
-		)
-		(pin "6"
-		)
 		(instances
 			(project "dual-sx1281-carrier-board"
 				(path "/dd3d82ed-b0ea-48bf-93b4-f28bcc2a961e"
-					(reference "U3")
+					(reference "J6")
 					(unit 1)
 				)
@@
 	)
 	(symbol
-		(lib_id "power:+3V3")
-		(at 54.61 154.94 0)
+		(lib_id "deets kicad lib:E28-2G4M20SX")
+		(at 246.38 66.04 0)
 		(unit 1)
 		(body_style 1)
@@
 		(dnp no)
 		(fields_autoplaced yes)
-		(property "Reference" "#PWR016"
-			(at 54.61 158.75 0)
-			(hide yes)
+		(property "Reference" "U3"
+			(at 248.5233 50.8 0)
 			(show_name no)
 			(do_not_autoplace no)
@@
 					(size 1.27 1.27)
 				)
+				(justify left)
 			)
 		)
-		(property "Value" "+3V3"
-			(at 54.61 149.86 0)
+		(property "Value" "E28-2G4M20SX"
+			(at 246.126 82.042 0)
+			(hide yes)
 			(show_name no)
 			(do_not_autoplace no)
@@
 			)
 		)
-		(property "Footprint" ""
-			(at 54.61 154.94 0)
+		(property "Footprint" "deets:E28-2G4M20SX"
+			(at 246.126 48.514 0)
 			(hide yes)
 			(show_name no)
@@
 		)
 		(property "Datasheet" ""
-			(at 54.61 154.94 0)
+			(at 246.38 66.04 0)
 			(hide yes)
 			(show_name no)
@@
 			)
 		)
-		(property "Description" "Power symbol creates a global label with name \"+3V3\""
-			(at 54.61 154.94 0)
+		(property "Description" "Lora1"
+			(at 248.5233 53.34 0)
+			(show_name no)
+			(do_not_autoplace no)
+			(effects
+				(font
+					(size 1.27 1.27)
+				)
+				(justify left)
+			)
+		)
+		(property "Manufacturer" "SenseCAP"
+			(at 246.126 51.054 0)
 			(hide yes)
 			(show_name no)
@@
 			)
 		)
+		(pin "15"
+		)
+		(pin "10"
+		)
+		(pin "12"
+		)
+		(pin "14"
+		)
+		(pin "13"
+		)
+		(pin "11"
+		)
+		(pin "2"
+		)
+		(pin "16"
+		)
+		(pin "7"
+		)
+		(pin "4"
+		)
+		(pin "3"
+		)
+		(pin "9"
+		)
 		(pin "1"
 		)
+		(pin "5"
+		)
+		(pin "8"
+		)
+		(pin "6"
+		)
 		(instances
 			(project "dual-sx1281-carrier-board"
 				(path "/dd3d82ed-b0ea-48bf-93b4-f28bcc2a961e"
-					(reference "#PWR016")
+					(reference "U3")
 					(unit 1)
 				)
@@
 	)
 	(symbol
-		(lib_id "Connector_Generic:Conn_01x05")
-		(at 111.76 134.62 0)
-		(mirror y)
+		(lib_id "power:+3V3")
+		(at 54.61 154.94 0)
 		(unit 1)
 		(body_style 1)
@@
 		(dnp no)
 		(fields_autoplaced yes)
-		(property "Reference" "J1"
-			(at 111.76 123.19 0)
+		(property "Reference" "#PWR016"
+			(at 54.61 158.75 0)
+			(hide yes)
 			(show_name no)
 			(do_not_autoplace no)
@@
 			)
 		)
-		(property "Value" "Conn_01x05"
-			(at 111.76 125.73 0)
+		(property "Value" "+3V3"
+			(at 54.61 149.86 0)
 			(show_name no)
 			(do_not_autoplace no)
@@
 			)
 		)
-		(property "Footprint" "Connector_Molex:Molex_PicoBlade_53398-0571_1x05-1MP_P1.25mm_Vertical"
-			(at 111.76 134.62 0)
+		(property "Footprint" ""
+			(at 54.61 154.94 0)
 			(hide yes)
 			(show_name no)
@@
 		)
 		(property "Datasheet" ""
-			(at 111.76 134.62 0)
+			(at 54.61 154.94 0)
 			(hide yes)
 			(show_name no)
@@
 			)
 		)
-		(property "Description" "Generic connector, single row, 01x05, script generated (kicad-library-utils/schlib/autogen/connector/)"
-			(at 111.76 134.62 0)
+		(property "Description" "Power symbol creates a global label with name \"+3V3\""
+			(at 54.61 154.94 0)
 			(hide yes)
 			(show_name no)
@@
 			)
 		)
-		(pin "4"
-		)
-		(pin "2"
-		)
 		(pin "1"
 		)
-		(pin "3"
-		)
-		(pin "5"
-		)
 		(instances
 			(project "dual-sx1281-carrier-board"
 				(path "/dd3d82ed-b0ea-48bf-93b4-f28bcc2a961e"
-					(reference "J1")
+					(reference "#PWR016")
 					(unit 1)
 				)

Commit message: Added DigiKey part numbers
Parts:
- D1: value LED -> RED; DigikeyPartNumber (none) -> 5962-XL-1608SURC-06TR-ND
- D2: value LED -> GREEN; DigikeyPartNumber (none) -> 5962-XL-1608UGC-04TR-ND
- D3: value LED -> BLUE; DigikeyPartNumber (none) -> 5962-XL-N1608SURUBCTR-ND
- J2, J3, J4, J5: now left out of the parts list
- J6: DigikeyPartNumber (none) -> WM7610CT-ND
- U1: DigikeyPartNumber (none) -> 2648-SC0914(13)CT-ND
- U2: DigikeyPartNumber (none) -> W25Q32JVSSIQ-ND

Commit message: Add digikey part numbers and a bit of silk screen tinkering
Parts:
- R1: DigikeyPartNumber (none) -> 541-10.0KLCT-ND
- R4: DigikeyPartNumber (none) -> 541-10.0KHCT-ND
- R5, R6, R7: DigikeyPartNumber (none) -> P300GCT-ND
Changed lines of the file:
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@@
 			)
 		)
-		(property "DigikeyPartNumber" ""
+		(property "DigikeyPartNumber" "P300GCT-ND"
 			(at 210.82 152.4 0)
 			(hide yes)
@@
 			)
 		)
-		(property "DigikeyPartNumber" ""
+		(property "DigikeyPartNumber" "541-10.0KHCT-ND"
 			(at 115.57 62.23 0)
 			(hide yes)
@@
 			)
 		)
-		(property "DigikeyPartNumber" ""
+		(property "DigikeyPartNumber" "P300GCT-ND"
 			(at 220.98 152.4 0)
 			(hide yes)
@@
 			)
 		)
-		(property "DigikeyPartNumber" ""
+		(property "DigikeyPartNumber" "541-10.0KLCT-ND"
 			(at 120.65 87.63 0)
 			(hide yes)
@@
 			)
 		)
-		(property "DigikeyPartNumber" ""
+		(property "DigikeyPartNumber" "P300GCT-ND"
 			(at 200.66 152.4 0)
 			(hide yes)
